Commit message: Update Equipo5.urdf
limites

File: Practicas/Practica1/Equipo5.urdf (robot description, URDF)
Before this commit: robot rrp_robot, 10 links, 9 joints
Joints:
- joint arm_joint: limit (none) -> lower=-3.14 upper=3.14 effort=10.0 velocity=0.5
- joint shoulder_joint: limit (none) -> lower=-3.14 upper=3.14 effort=10.0 velocity=0.5

Commit message: Update Equipo5.urdf
mejora

File: Practicas/Practica1/Equipo5.urdf (robot description, URDF)
Before this commit: robot rrp_robot, 10 links, 9 joints
Joints:
- joint arm_joint: origin xyz=0 0.3 0 rpy=0 0 0 -> xyz=0 0.275 0.025 rpy=0 0 0
